File: Kicad/romcart/v1a/v1a.kicad_pcb (KiCad board)
At the start: 2 copper layers, 56.9 x 38.6 mm, 6 parts, among them J1 Conn_02x22_Odd_Even, U1 SST39SF040

Commit message: update kicad files
Other:
- board text added: "Designed January 2024 by smal smaldragon.github.io"
- board text removed: "Designed November 2023 by smal smaldragon.github.io"
Changed lines of the file:
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@@
     (effects (font (size 1 1) (thickness 0.15)) (justify left bottom mirror))
   )
-  (gr_text "Designed November 2023\nby smal\nsmaldragon.github.io" (at 96.52 62.23) (layer "B.SilkS")
+  (gr_text "Designed January 2024\nby smal\nsmaldragon.github.io" (at 96.52 62.23) (layer "B.SilkS")
     (effects (font (size 1 1) (thickness 0.15)) (justify left bottom mirror))
   )
@@
     (effects (font (size 2 2) (thickness 0.4) bold) (justify bottom))
   )
-  (gr_text "v1a" (at 70.7136 62.1538) (layer "F.SilkS")
+  (gr_text "v1a" (at 71.882 60.96) (layer "F.SilkS")
     (effects (font (size 1 1) (thickness 0.15)) (justify bottom))
   )
