File: Kicad/ramcart/v1a/v1a.kicad_sch (KiCad schematic)
At the start: 8 parts, among them J1 Conn_02x22_Odd_Even, U1 AS6C4008-55PCN

Commit message: big v1b commit
Connections:
- net +5V: no longer JP1.3 (B), U1.24 (OE#)
- net B6: now also JP1.3 (B)
- net GND: now also U1.24 (OE#)
Changed lines of the file:
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@@
+    (stroke (width 0) (type default))
+  )
+  (wire (pts (xy 68.58 60.96) (xy 62.23 60.96))
     (stroke (width 0) (type default))
   )
@@
     )
   )
+  (global_label "B6" (shape input) (at 24.13 71.12 90) (fields_autoplaced)
+    (effects (font (size 1.27 1.27)) (justify left))
+    (property "Intersheetrefs" "${INTERSHEET_REFS}" (at 24.13 65.6553 90)
+      (effects (font (size 1.27 1.27)) (justify left) hide)
+    )
+  )
   (global_label "B2" (shape output) (at 153.67 46.99 90) (fields_autoplaced)
     (effects (font (size 1.27 1.27)) (justify left))
@@
     (property "Intersheetrefs" "${INTERSHEET_REFS}" (at 31.5467 38.1 0)
       (effects (font (size 1.27 1.27)) (justify right) hide)
+    )
+  )
+  (symbol (lib_id "power:GND") (at 68.58 60.96 90) (unit 1)
+    (in_bom yes) (on_board yes) (dnp no) (fields_autoplaced)
+    (property "Reference" "#PWR08" (at 74.93 60.96 0)
+      (effects (font (size 1.27 1.27)) hide)
+    )
+    (property "Value" "GND" (at 72.39 60.96 90)
+      (effects (font (size 1.27 1.27)) (justify right))
+    )
+    (property "Footprint" "" (at 68.58 60.96 0)
+      (effects (font (size 1.27 1.27)) hide)
+    )
+    (property "Datasheet" "" (at 68.58 60.96 0)
+      (effects (font (size 1.27 1.27)) hide)
+    )
+    (pin "1")
+    (instances
+      (project "v1a"
+        (path "/b7e521a9-0c53-40c9-9596-7011d46f246c"
+          (reference "#PWR08") (unit 1)
+        )
+      )
     )
   )
@@
     )
   )
-  (symbol (lib_id "power:+5V") (at 62.23 60.96 270) (unit 1)
-    (in_bom yes) (on_board yes) (dnp no) (fields_autoplaced)
-    (property "Reference" "#PWR09" (at 58.42 60.96 0)
-      (effects (font (size 1.27 1.27)) hide)
-    )
-    (property "Value" "+5V" (at 67.31 60.96 0)
-      (effects (font (size 1.27 1.27)) hide)
-    )
-    (property "Footprint" "" (at 62.23 60.96 0)
-      (effects (font (size 1.27 1.27)) hide)
-    )
-    (property "Datasheet" "" (at 62.23 60.96 0)
-      (effects (font (size 1.27 1.27)) hide)
-    )
-    (pin "1")
-    (instances
-      (project "v1a"
-        (path "/b7e521a9-0c53-40c9-9596-7011d46f246c"
-          (reference "#PWR09") (unit 1)
-        )
-      )
-    )
-  )
   (symbol (lib_id "power:+5V") (at 49.53 22.86 270) (unit 1)
     (in_bom yes) (on_board yes) (dnp no) (fields_autoplaced)
@@
         )
       )
-    )
-  )
-  (symbol (lib_id "power:+5V") (at 24.13 71.12 0) (unit 1)
-    (in_bom yes) (on_board yes) (dnp no) (fields_autoplaced)
-    (property "Reference" "#PWR010" (at 24.13 74.93 0)
-      (effects (font (size 1.27 1.27)) hide)
-    )
-    (property "Value" "+5V" (at 24.13 66.04 0)
-      (effects (font (size 1.27 1.27)))
-    )
-    (property "Footprint" "" (at 24.13 71.12 0)
-      (effects (font (size 1.27 1.27)) hide)
-    )
-    (property "Datasheet" "" (at 24.13 71.12 0)
-      (effects (font (size 1.27 1.27)) hide)
-    )
-    (pin "1")
-    (instances
-      (project "v1a"
-        (path "/b7e521a9-0c53-40c9-9596-7011d46f246c"
-          (reference "#PWR010") (unit 1)
-        )
-      )
