File: Kicad/case/back/back.kicad_pcb (KiCad board)
At the start: 2 copper layers, 237.2 x 31.5 mm, 2 parts

Commit message: v2a update
Parts:
- added REF**: CenterPositiveSymbol, Smal:CenterPositiveSymbol, F.Cu at (33.9, 111.0)
Other:
- outline, holes or cut-outs redrawn
- board text added: "5v"
- board text added: "LINE"
- board text added: "RGB"
- board text added: "SLOT 1"
- board text added: "SLOT 2"
- board text removed: "5V"
- board text removed: "AUX"
- board text removed: "CARTRIDGE 1"
- board text removed: "CARTRIDGE 2"
- board text removed: "SCART"
