File: Kicad/mainboard/v1a/video.kicad_sch (KiCad schematic)
At the start: 30 parts, among them U10 74HC590A, U11 74HC590A, U12 74HC574, U13 74HC165, U14 74HC157, U15 74HC574, U7 74HC138, U8 SST39SF, U9 74HC574

Commit message: big v1b commit
Parts:
- added J?: DE15_Plug_HighDensity_MountingHoles, Connector_Dsub:DSUB-15-HD_Female_Horizontal_P2.29x1.98mm_EdgePinOffset3.03mm_Housed_MountingHolesOffset4.94mm, symbol Connector:DE15_Plug_HighDensity_MountingHoles
Changed lines of the file:
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@@
+    )
+  )
+  (symbol (lib_id "Connector:DE15_Plug_HighDensity_MountingHoles") (at 34.29 111.76 0) (unit 1)
+    (in_bom yes) (on_board yes) (dnp no) (fields_autoplaced)
+    (property "Reference" "J?" (at 34.29 88.9 0)
+      (effects (font (size 1.27 1.27)))
+    )
+    (property "Value" "DE15_Plug_HighDensity_MountingHoles" (at 34.29 91.44 0)
+      (effects (font (size 1.27 1.27)))
+    )
+    (property "Footprint" "Connector_Dsub:DSUB-15-HD_Female_Horizontal_P2.29x1.98mm_EdgePinOffset3.03mm_Housed_MountingHolesOffset4.94mm" (at 10.16 101.6 0)
+      (effects (font (size 1.27 1.27)) hide)
+    )
+    (property "Datasheet" " ~" (at 10.16 101.6 0)
+      (effects (font (size 1.27 1.27)) hide)
+    )
+    (pin "8")
+    (pin "3")
+    (pin "6")
+    (pin "7")
+    (pin "9")
+    (pin "2")
+    (pin "4")
+    (pin "1")
+    (pin "0")
+    (pin "13")
+    (pin "12")
+    (pin "5")
+    (pin "11")
+    (pin "14")
+    (pin "15")
+    (pin "10")
+    (instances
+      (project "v1a"
+        (path "/82bc3382-6295-4121-a2db-2433a00f189b/08a65c83-f6b0-43c9-8af0-6a881bb0b65a"
+          (reference "J?") (unit 1)
+        )
+      )
     )
   )

Commit message: v2a update
Parts:
- gave numbers to parts that had none: 1
Changed lines of the file:
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@@
   (symbol (lib_id "Connector:DE15_Plug_HighDensity_MountingHoles") (at 34.29 111.76 0) (unit 1)
     (in_bom yes) (on_board yes) (dnp no) (fields_autoplaced)
-    (property "Reference" "J?" (at 34.29 88.9 0)
+    (property "Reference" "J7" (at 34.29 88.9 0)
       (effects (font (size 1.27 1.27)))
     )
@@
       (project "v1a"
         (path "/82bc3382-6295-4121-a2db-2433a00f189b/08a65c83-f6b0-43c9-8af0-6a881bb0b65a"
-          (reference "J?") (unit 1)
+          (reference "J7") (unit 1)
         )
       )
