File: Kicad/keyboard/keyboard/keyboard.kicad_pcb (KiCad board)
At the start: 2 copper layers, 239.3 x 76 mm, 89 parts, among them J1 Conn_01x05_Pin, J2 Conn_01x08_Pin, SW1 ESC, SW10 Q, SW11 S, SW12 G, SW13 Y, SW14 J, SW15 K, SW16 P, SW17 Shift, SW18 A, SW19 D, SW2 W, SW20 V, SW21 H, SW22 M, SW23 L, SW24 BackSpace, SW25 Menu, SW26 Z, SW27 F, SW28 B, SW29 N, SW3 E, SW30 ||, SW31 ., SW32 Enter, SW33 Ctrl, SW34 X, SW35 C, SW36 Space, SW37 Up, SW38 Left, SW39 Down, SW4 R, SW40 Right, SW5 T, SW6 U, SW7 I, SW8 O, SW9 Alt

Commit message: v2a update
Parts:
- removed D41, D42, D43, D44, D45: 1N4148, Diode_THT:D_DO-35_SOD27_P7.62mm_Horizontal
- S1: footprint PCM_marbastlib-mx:STAB_MX_P_2u -> KS27_PCB_STAB:ks27_2u_pcb_cherry_plate_stab
- S2: footprint PCM_marbastlib-mx:STAB_MX_P_6.25u -> KS27_PCB_STAB:ks26_6.25u_pcb_cherry_plate
- SW1, SW10, SW11, SW12, SW13, SW14, SW15, SW16, SW18, SW19, SW2, SW20, SW21, SW22, SW23, SW26, SW27, SW28, SW29, SW3, SW34, SW35, SW4, SW5, SW6, SW7, SW8: footprint keyswitches.pretty-2.1:SW_PG1350_MX_Hybrid -> SMAL:SW_Redragon_LowProfile_PCB_1.00u
- SW17: value Shift -> SHIFT; footprint keyswitches.pretty-2.1:SW_PG1350_MX_Hybrid -> SMAL:SW_Redragon_LowProfile_PCB_1.75u
- SW24: value BackSpace -> DELETE; footprint keyswitches.pretty-2.1:SW_PG1350_MX_Hybrid -> SMAL:SW_Redragon_LowProfile_PCB_1.25u
- SW25: value Menu -> MENU; footprint keyswitches.pretty-2.1:SW_PG1350_MX_Hybrid -> SMAL:SW_Redragon_LowProfile_PCB_1.75u
- SW30: footprint keyswitches.pretty-2.1:SW_PG1350_MX_Hybrid -> SMAL:SW_Redragon_LowProfile_PCB_1.50u
- SW31: value . -> ..; footprint keyswitches.pretty-2.1:SW_PG1350_MX_Hybrid -> SMAL:SW_Redragon_LowProfile_PCB_1.00u
- SW32: value Enter -> ENTER; footprint keyswitches.pretty-2.1:SW_PG1350_MX_Hybrid -> SMAL:SW_Redragon_LowProfile_PCB_2.00u
- SW33: value Ctrl -> CTRL; footprint keyswitches.pretty-2.1:SW_PG1350_MX_Hybrid -> SMAL:SW_Redragon_LowProfile_PCB_1.25u
- SW36: value Space -> SPACE; footprint keyswitches.pretty-2.1:SW_PG1350_MX_Hybrid -> SMAL:SW_Redragon_LowProfile_PCB_6.25u
- SW37: value Up -> UP; footprint keyswitches.pretty-2.1:SW_PG1350_MX_Hybrid -> SMAL:SW_Redragon_LowProfile_PCB_1.00u
- SW38: value Left -> LEFT; footprint keyswitches.pretty-2.1:SW_PG1350_MX_Hybrid -> SMAL:SW_Redragon_LowProfile_PCB_1.00u
- SW39: value Down -> DOWN; footprint keyswitches.pretty-2.1:SW_PG1350_MX_Hybrid -> SMAL:SW_Redragon_LowProfile_PCB_1.00u
- SW40: value Right -> RIGHT; footprint keyswitches.pretty-2.1:SW_PG1350_MX_Hybrid -> SMAL:SW_Redragon_LowProfile_PCB_1.00u
- SW9: value Alt -> ALT; footprint keyswitches.pretty-2.1:SW_PG1350_MX_Hybrid -> SMAL:SW_Redragon_LowProfile_PCB_1.25u
- moved D9 169.5 mm to (47.5, 62.7)
- moved D18 168.3 mm to (68.9, 62.7)
- moved D38 167.5 mm to (220.9, 100.7)
- moved D17 150.9 mm to (52.2, 81.7)
- moved D39 148.4 mm to (239.9, 100.7)
- moved D26 143.8 mm to (78.4, 81.7)
- moved D30 142.5 mm to (216.1, 81.7)
- moved D40 142.1 mm to (253.2, 95.0), turned to 180 degrees
- moved D27 132.1 mm to (125.9, 62.7)
- moved D33 123.0 mm to (47.5, 100.7)
- moved D37 120.9 mm to (220.9, 81.7), turned to -90 degrees
- moved D35 119.8 mm to (116.4, 81.7), turned to -90 degrees
- moved D34 117.3 mm to (97.4, 81.7)
- moved D25 116.0 mm to (76.0, 100.7)
- moved D31 108.6 mm to (234.2, 57.0), turned to 180 degrees
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Connections:
- D1 pad 1: /Row 0 -> Net-(D1-K)
- D1 pad 2: Net-(D1-A) -> /Col 0
- D10 pad 1: /Row 1 -> Net-(D10-K)
- D10 pad 2: Net-(D10-A) -> /Col 1
- D11 pad 2: /Col 0 -> /Col 2
- D12 pad 2: /Col 1 -> /Col 3
- D13 pad 2: /Col 2 -> /Col 4
- D14 pad 2: /Col 3 -> /Col 5
- D15 pad 2: /Col 4 -> /Col 6
- D16 pad 2: /Col 5 -> /Col 7
- D17 pad 2: /Col 6 -> /Col 0
- D18 pad 2: /Col 7 -> /Col 1
- D19 pad 1: /Row 2 -> Net-(D19-K)
- D19 pad 2: Net-(D19-A) -> /Col 2
- D2 pad 2: /Col 0 -> /Col 1
- D20 pad 2: /Col 0 -> /Col 3
- D21 pad 2: /Col 1 -> /Col 4
- D22 pad 2: /Col 2 -> /Col 5
- D23 pad 2: /Col 3 -> /Col 6
- D24 pad 2: /Col 4 -> /Col 7
- D25 pad 2: /Col 5 -> /Col 0
- D26 pad 2: /Col 6 -> /Col 1
- D27 pad 2: /Col 7 -> /Col 2
- D28 pad 1: /Row 3 -> Net-(D28-K)
- D28 pad 2: Net-(D28-A) -> /Col 3
- D29 pad 2: /Col 0 -> /Col 4
- D3 pad 2: /Col 1 -> /Col 2
- D30 pad 2: /Col 1 -> /Col 5
- D31 pad 2: /Col 2 -> /Col 6
- D32 pad 2: /Col 3 -> /Col 7
- D33 pad 2: /Col 4 -> /Col 0
- D34 pad 2: /Col 5 -> /Col 1
- D35 pad 2: /Col 6 -> /Col 2
- D36 pad 2: /Col 7 -> /Col 3
- D37 pad 1: /Row 4 -> Net-(D37-K)
- D37 pad 2: Net-(D37-A) -> /Col 4
- D38 pad 2: /Col 0 -> /Col 5
- D39 pad 2: /Col 1 -> /Col 6
- D4 pad 2: /Col 2 -> /Col 3
- D40 pad 2: /Col 2 -> /Col 7
- D5 pad 2: /Col 3 -> /Col 4
- D6 pad 2: /Col 4 -> /Col 5
- D7 pad 2: /Col 5 -> /Col 6
- D8 pad 2: /Col 6 -> /Col 7
- D9 pad 2: /Col 7 -> /Col 0
- SW1 pad 1: Net-(D1-A) -> /Row 0
- SW1 pad 2: Net-(D2-K) -> Net-(D1-K)
- SW10 pad 1: Net-(D10-A) -> /Row 1
- SW10 pad 2: Net-(D12-K) -> Net-(D10-K)
- SW11 pad 1: Net-(D10-A) -> /Row 1
- SW11 pad 2: Net-(D13-K) -> Net-(D11-K)
- SW12 pad 1: Net-(D10-A) -> /Row 1
- SW12 pad 2: Net-(D14-K) -> Net-(D12-K)
- SW13 pad 1: Net-(D10-A) -> /Row 1
- SW13 pad 2: Net-(D15-K) -> Net-(D13-K)
- SW14 pad 1: Net-(D10-A) -> /Row 1
- SW14 pad 2: Net-(D16-K) -> Net-(D14-K)
- SW15 pad 1: Net-(D10-A) -> /Row 1
- SW15 pad 2: Net-(D17-K) -> Net-(D15-K)
- SW16 pad 1: Net-(D10-A) -> /Row 1
- SW16 pad 2: Net-(D18-K) -> Net-(D16-K)
- SW17 pad 1: Net-(D19-A) -> /Row 2
- SW17 pad 2: Net-(D20-K) -> Net-(D17-K)
- SW18 pad 1: Net-(D19-A) -> /Row 2
- SW18 pad 2: Net-(D21-K) -> Net-(D18-K)
- SW19 pad 1: Net-(D19-A) -> /Row 2
- SW19 pad 2: Net-(D22-K) -> Net-(D19-K)
- SW2 pad 1: Net-(D1-A) -> /Row 0
- SW2 pad 2: Net-(D3-K) -> Net-(D2-K)
- SW20 pad 1: Net-(D19-A) -> /Row 2
- SW20 pad 2: Net-(D23-K) -> Net-(D20-K)
- SW21 pad 1: Net-(D19-A) -> /Row 2
- SW21 pad 2: Net-(D24-K) -> Net-(D21-K)
- SW22 pad 1: Net-(D19-A) -> /Row 2
- SW22 pad 2: Net-(D25-K) -> Net-(D22-K)
- SW23 pad 1: Net-(D19-A) -> /Row 2
- SW23 pad 2: Net-(D26-K) -> Net-(D23-K)
- SW24 pad 1: Net-(D19-A) -> /Row 2
- SW24 pad 2: Net-(D27-K) -> Net-(D24-K)
- SW25 pad 1: Net-(D28-A) -> /Row 3
- SW25 pad 2: Net-(D29-K) -> Net-(D25-K)
- SW26 pad 1: Net-(D28-A) -> /Row 3
- SW26 pad 2: Net-(D30-K) -> Net-(D26-K)
- SW27 pad 1: Net-(D28-A) -> /Row 3
- SW27 pad 2: Net-(D31-K) -> Net-(D27-K)
- SW28 pad 1: Net-(D28-A) -> /Row 3
- SW28 pad 2: Net-(D32-K) -> Net-(D28-K)
- SW29 pad 1: Net-(D28-A) -> /Row 3
- SW29 pad 2: Net-(D33-K) -> Net-(D29-K)
- SW3 pad 1: Net-(D1-A) -> /Row 0
- SW3 pad 2: Net-(D4-K) -> Net-(D3-K)
- SW30 pad 1: Net-(D28-A) -> /Row 3
- SW30 pad 2: Net-(D34-K) -> Net-(D30-K)
- SW31 pad 1: Net-(D28-A) -> /Row 3
- SW31 pad 2: Net-(D35-K) -> Net-(D31-K)
- SW32 pad 1: Net-(D28-A) -> /Row 3
- SW32 pad 2: Net-(D36-K) -> Net-(D32-K)
- SW33 pad 1: Net-(D37-A) -> /Row 4
- SW33 pad 2: Net-(D38-K) -> Net-(D33-K)
- SW34 pad 1: Net-(D37-A) -> /Row 4
- SW34 pad 2: Net-(D39-K) -> Net-(D34-K)
- SW35 pad 1: Net-(D37-A) -> /Row 4
- SW35 pad 2: Net-(D40-K) -> Net-(D35-K)
- SW36 pad 1: Net-(D37-A) -> /Row 4
- SW36 pad 2: Net-(D41-K) -> Net-(D36-K)
- SW37 pad 1: Net-(D37-A) -> /Row 4
- SW37 pad 2: Net-(D42-K) -> Net-(D37-K)
- SW38 pad 1: Net-(D37-A) -> /Row 4
- SW38 pad 2: Net-(D43-K) -> Net-(D38-K)
- SW39 pad 1: Net-(D37-A) -> /Row 4
- SW39 pad 2: Net-(D44-K) -> Net-(D39-K)
- SW4 pad 1: Net-(D1-A) -> /Row 0
- SW4 pad 2: Net-(D5-K) -> Net-(D4-K)
- SW40 pad 1: Net-(D37-A) -> /Row 4
- SW40 pad 2: Net-(D45-K) -> Net-(D40-K)
- SW5 pad 1: Net-(D1-A) -> /Row 0
- SW5 pad 2: Net-(D6-K) -> Net-(D5-K)
- SW6 pad 1: Net-(D1-A) -> /Row 0
- SW6 pad 2: Net-(D7-K) -> Net-(D6-K)
- SW7 pad 1: Net-(D1-A) -> /Row 0
- SW7 pad 2: Net-(D8-K) -> Net-(D7-K)
- SW8 pad 1: Net-(D1-A) -> /Row 0
- SW8 pad 2: Net-(D9-K) -> Net-(D8-K)
- SW9 pad 1: Net-(D10-A) -> /Row 1
- SW9 pad 2: Net-(D11-K) -> Net-(D9-K)
Routing:
- net Net-(D10-A): track 409.5 -> 0.00 mm
- net Net-(D19-A): track 405.0 -> 0.00 mm
- net Net-(D37-A): track 355.1 -> 0.00 mm
- net Net-(D28-A): track 350.1 -> 0.00 mm
- net /Row 1: track 21.0 -> 355.7 mm
- net /Row 2: track 21.1 -> 351.6 mm
- net Net-(D1-A): track 318.2 -> 0.00 mm
- net /Row 4: track 19.4 -> 294.1 mm
- net /Row 3: track 21.1 -> 292.1 mm
- net /Row 0: track 19.4 -> 267.7 mm
- net /Col 4: track 153.2 -> 205.2 mm
- net /Col 6: track 230.2 -> 195.8 mm
- net Net-(D42-K): track 25.7 -> 0.00 mm
- net Net-(D43-K): track 23.9 -> 0.00 mm
- net Net-(D41-K): track 23.6 -> 0.00 mm
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Other:
- board text added: "JLCJLCJLCJLC"

Commit message: Update board files
Parts:
- J1: value Conn_01x05_Pin -> Conn_01x06_Pin; footprint Connector_PinHeader_2.54mm:PinHeader_1x05_P2.54mm_Vertical -> Connector_PinHeader_2.54mm:PinHeader_1x06_P2.54mm_Vertical
- S1: footprint KS27_PCB_STAB:ks27_2u_pcb_cherry_plate_stab -> ks27_pcb_stab:ks27_2u_pcb_cherry_plate_stab
- S2: footprint KS27_PCB_STAB:ks26_6.25u_pcb_cherry_plate -> ks27_pcb_stab:ks26_6.25u_pcb_cherry_plate
- SW1, SW10, SW11, SW12, SW13, SW14, SW15, SW16, SW18, SW19, SW2, SW20, SW21, SW22, SW23, SW26, SW27, SW28, SW29, SW3, SW31, SW34, SW35, SW37, SW38, SW39, SW4, SW40, SW5, SW6, SW7, SW8: footprint SMAL:SW_Redragon_LowProfile_PCB_1.00u -> Smal:SW_Redragon_LowProfile_PCB_1.00u
- SW17: footprint SMAL:SW_Redragon_LowProfile_PCB_1.75u -> Smal:SW_Redragon_LowProfile_PCB_1.75u
- SW24: value DELETE -> BACK; footprint SMAL:SW_Redragon_LowProfile_PCB_1.25u -> Smal:SW_Redragon_LowProfile_PCB_1.25u
- SW25: footprint SMAL:SW_Redragon_LowProfile_PCB_1.75u -> Smal:SW_Redragon_LowProfile_PCB_1.50u
- SW30: footprint SMAL:SW_Redragon_LowProfile_PCB_1.50u -> Smal:SW_Redragon_LowProfile_PCB_1.50u
- SW32: footprint SMAL:SW_Redragon_LowProfile_PCB_2.00u -> Smal:SW_Redragon_LowProfile_PCB_2.00u
- SW33: footprint SMAL:SW_Redragon_LowProfile_PCB_1.25u -> Smal:SW_Redragon_LowProfile_PCB_1.50u
- SW36: footprint SMAL:SW_Redragon_LowProfile_PCB_6.25u -> Smal:SW_Redragon_LowProfile_PCB_6.25u
- SW9: footprint SMAL:SW_Redragon_LowProfile_PCB_1.25u -> Smal:SW_Redragon_LowProfile_PCB_1.25u
- moved J2 17.8 mm to (175.2, 108.0), turned to 90 degrees
- moved D25 2.38 mm to (78.4, 100.7)
- moved D33 2.38 mm to (49.9, 100.7)
- moved SW25 2.38 mm to (68.9, 104.5)
- moved SW33 2.38 mm to (40.4, 104.5)
- moved D36 2.18 mm to (152.0, 102.9)
Connections:
- D1 pad 2: /Col 0 -> /Col 7
- D10 pad 2: /Col 1 -> /Col 6
- D11 pad 2: /Col 2 -> /Col 5
- D12 pad 2: /Col 3 -> /Col 4
- D13 pad 2: /Col 4 -> /Col 3
- D14 pad 2: /Col 5 -> /Col 2
- D15 pad 2: /Col 6 -> /Col 1
- D16 pad 2: /Col 7 -> /Col 0
- D17 pad 2: /Col 0 -> /Col 7
- D18 pad 2: /Col 1 -> /Col 6
- D19 pad 2: /Col 2 -> /Col 5
- D2 pad 2: /Col 1 -> /Col 6
- D20 pad 2: /Col 3 -> /Col 4
- D21 pad 2: /Col 4 -> /Col 3
- D22 pad 2: /Col 5 -> /Col 2
- D23 pad 2: /Col 6 -> /Col 1
- D24 pad 2: /Col 7 -> /Col 0
- D25 pad 2: /Col 0 -> /Col 7
- D26 pad 2: /Col 1 -> /Col 6
- D27 pad 2: /Col 2 -> /Col 5
- D28 pad 2: /Col 3 -> /Col 4
- D29 pad 2: /Col 4 -> /Col 3
- D3 pad 2: /Col 2 -> /Col 5
- D30 pad 2: /Col 5 -> /Col 2
- D31 pad 2: /Col 6 -> /Col 1
- D32 pad 2: /Col 7 -> /Col 0
- D33 pad 2: /Col 0 -> /Col 7
- D34 pad 2: /Col 1 -> /Col 6
- D35 pad 2: /Col 2 -> /Col 5
- D36 pad 2: /Col 3 -> /Col 4
- D37 pad 2: /Col 4 -> /Col 3
- D38 pad 2: /Col 5 -> /Col 2
- D39 pad 2: /Col 6 -> /Col 1
- D4 pad 2: /Col 3 -> /Col 4
- D40 pad 2: /Col 7 -> /Col 0
- D5 pad 2: /Col 4 -> /Col 3
- D6 pad 2: /Col 5 -> /Col 2
- D7 pad 2: /Col 6 -> /Col 1
- D8 pad 2: /Col 7 -> /Col 0
- D9 pad 2: /Col 0 -> /Col 7
- J1 pad 1: /Row 0 -> /Row 4
- J1 pad 2: /Row 1 -> /Row 3
- J1 pad 4: /Row 3 -> /Row 1
- J1 pad 5: /Row 4 -> /Row 0
- SW1 pad 1: /Row 0 -> /Row 4
- SW10 pad 1: /Row 1 -> /Row 3
- SW11 pad 1: /Row 1 -> /Row 3
- SW12 pad 1: /Row 1 -> /Row 3
- SW13 pad 1: /Row 1 -> /Row 3
- SW14 pad 1: /Row 1 -> /Row 3
- SW15 pad 1: /Row 1 -> /Row 3
- SW16 pad 1: /Row 1 -> /Row 3
- SW2 pad 1: /Row 0 -> /Row 4
- SW25 pad 1: /Row 3 -> /Row 1
- SW26 pad 1: /Row 3 -> /Row 1
- SW27 pad 1: /Row 3 -> /Row 1
- SW28 pad 1: /Row 3 -> /Row 1
- SW29 pad 1: /Row 3 -> /Row 1
- SW3 pad 1: /Row 0 -> /Row 4
- SW30 pad 1: /Row 3 -> /Row 1
- SW31 pad 1: /Row 3 -> /Row 1
- SW32 pad 1: /Row 3 -> /Row 1
- SW33 pad 1: /Row 4 -> /Row 0
- SW34 pad 1: /Row 4 -> /Row 0
- SW35 pad 1: /Row 4 -> /Row 0
- SW36 pad 1: /Row 4 -> /Row 0
- SW37 pad 1: /Row 4 -> /Row 0
- SW38 pad 1: /Row 4 -> /Row 0
- SW39 pad 1: /Row 4 -> /Row 0
- SW4 pad 1: /Row 0 -> /Row 4
- SW40 pad 1: /Row 4 -> /Row 0
- SW5 pad 1: /Row 0 -> /Row 4
- SW6 pad 1: /Row 0 -> /Row 4
- SW7 pad 1: /Row 0 -> /Row 4
- SW8 pad 1: /Row 0 -> /Row 4
- SW9 pad 1: /Row 1 -> /Row 3
Routing:
- net /Col 4: track 205.2 -> 126.8 mm
- net /Col 3: track 128.3 -> 205.2 mm
- net /Row 1: track 355.7 -> 291.1 mm
- net /Row 3: track 292.1 -> 356.3 mm
- net /Row 4: track 294.1 -> 267.7 mm
- net /Col 5: track 141.8 -> 168.1 mm
- net /Col 2: track 168.1 -> 141.8 mm
- net /Row 0: track 267.7 -> 291.9 mm
- net /Col 1: track 183.9 -> 197.2 mm
- net /Col 6: track 195.8 -> 183.9 mm
- net /Col 7: track 210.3 -> 201.8 mm
- net /Col 0: track 205.1 -> 210.7 mm
- net Net-(D40-K): track 20.7 -> 17.5 mm
- net Net-(D36-K): track 14.9 -> 13.9 mm
- net GND: vias 0 -> 17
- added copper zone on B.Cu, net GND
- added copper zone on F.Cu, net GND
- removed copper zone on B.Cu, net (none)
- removed copper zone on F.Cu, net (none)
Other:
- board size 239.3 x 76 mm -> 240.2 x 76 mm
- board text added: "C0"
- board text added: "C1"
- board text added: "C2"
- board text added: "C3"
- board text added: "C4"
- board text added: "C5"
- board text added: "C6"
- board text added: "C7"
- board text added: "GND"
- board text added: "R0"
- board text added: "R1"
- board text added: "R2"
- board text added: "R3"
- board text added: "R4"
