File: Kicad/mainboard/v1b/ClockReset.kicad_sch (KiCad schematic)
At the start: 21 parts, among them SW1 RESET, U2 74HC14, U3 74HC4520, U4 74HC4040, U5 SST39SF, U6 74HC574, Y1 12 Mhz

Commit message: big v1b commit
Parts:
- removed JP2: SolderJumper_3_Bridged12, Jumper:SolderJumper-3_P1.3mm_Bridged12_Pad1.0x1.5mm, symbol Jumper:SolderJumper_3_Bridged12
- removed U3: 74HC4520, PCM_Package_DIP_AKL:DIP-16_W7.62mm_Socket_LongPads, symbol 4xxx:4520
- added D6: D_Small, Diode_THT:D_DO-34_SOD68_P7.62mm_Horizontal, symbol Device:D_Small
- added R43: 3.3kΩ, Resistor_THT:R_Axial_DIN0204_L3.6mm_D1.6mm_P7.62mm_Horizontal, symbol Device:R_Small
- added U3: 74HC590, PCM_Package_DIP_AKL:DIP-16_W7.62mm_Socket_LongPads, symbol 74xx:74HC590
Connections:
- net ~{VPixel} is gone; now on net ~{VSync}: U6.13 (Q6)
- net +5V: now also R43.2, U3.10 (~{MRC}), U3.16 (VCC)
- net 12M: now also U3.11 (CPC), U3.13 (CPR)
- net 1M: now also U3.2 (Q2)
- net 3M: now also U3.1 (Q1)
- net 6M: now also U3.15 (Q0)
- net 750K: now also U3.3 (Q3)
- net AudioMux0: now also U3.4 (Q4)
- net AudioMux1: now also U3.5 (Q5)
- net GND: now also U3.12 (~{CE}), U3.14 (~{OE}), U3.8 (GND)
- net ~{RESET}: now also D6.2 (A), R43.1; no longer U2.6
- net ~{VSync}: no longer U6.14 (Q5)
- net at U4.10 (CLK): now also U3.9 (~{RCO}); no longer U5.9 (A3)
- net at U5.10 (A2): now also U3.6 (Q6)
- net VIrq renamed ~{HSync}
- new net: D6.1 (K), U2.6
- new net: U3.7 (Q7), U5.9 (A3)
- new net ~{Sync}: U6.14 (Q5)
Other:
- moved on the sheet: U5
