File: Kicad/mainboard/v1b/audio.kicad_sch (KiCad schematic)
At the start: 39 parts, among them U16 74HC139, U17 74HC153, U18 74HC670, U19 74HC670, U20 82C54, U21 82C54 (PLCC), U22 74HC165, U23 74HC165, U24 74HC165, U25 74HC165

Commit message: big v1b commit
Parts:
- R19, R20, R21, R22, R23, R28, R29, R30, R31, R32: value R2 -> 20KΩ
- R24, R25, R26, R33, R34, R35: value R1 -> 10KΩ
Connections:
- net volume: no longer U18.12 (~{Ew}), U19.12 (~{Ew})
- net ~{VolWr}: now also U18.12 (~{Ew}), U19.12 (~{Ew})
Changed lines of the file:
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@@
     (effects (font (size 1.27 1.27)) (justify left bottom))
-  )
-  (label "volume" (at 135.89 50.8 180) (fields_autoplaced)
-    (effects (font (size 1.27 1.27)) (justify right bottom))
   )
   (label "Osc 1" (at 29.21 181.61 180) (fields_autoplaced)
@@
   (label "volume" (at 60.96 50.8 0) (fields_autoplaced)
     (effects (font (size 1.27 1.27)) (justify left bottom))
-  )
-  (label "volume" (at 176.53 50.8 180) (fields_autoplaced)
-    (effects (font (size 1.27 1.27)) (justify right bottom))
   )
   (label "Ch2" (at 90.17 153.67 0) (fields_autoplaced)
@@
     )
   )
+  (global_label "~{VolWr}" (shape input) (at 176.53 50.8 180) (fields_autoplaced)
+    (effects (font (size 1.27 1.27)) (justify right))
+    (property "Intersheetrefs" "${INTERSHEET_REFS}" (at 168.4044 50.8 0)
+      (effects (font (size 1.27 1.27)) (justify right) hide)
+    )
+  )
   (global_label "D7" (shape input) (at 138.43 172.72 180) (fields_autoplaced)
     (effects (font (size 1.27 1.27)) (justify right))
@@
     (effects (font (size 1.27 1.27)) (justify right))
     (property "Intersheetrefs" "${INTERSHEET_REFS}" (at 117.06 125.73 0)
+      (effects (font (size 1.27 1.27)) (justify right) hide)
+    )
+  )
+  (global_label "~{VolWr}" (shape input) (at 135.89 50.8 180) (fields_autoplaced)
+    (effects (font (size 1.27 1.27)) (justify right))
+    (property "Intersheetrefs" "${INTERSHEET_REFS}" (at 127.7644 50.8 0)
       (effects (font (size 1.27 1.27)) (justify right) hide)
     )
@@
       (effects (font (size 1.27 1.27)))
     )
-    (property "Value" "R2" (at 198.12 100.33 90)
+    (property "Value" "20KΩ" (at 198.12 100.33 90)
       (effects (font (size 1.27 1.27)))
     )
@@
       (effects (font (size 1.27 1.27)) (justify right))
     )
-    (property "Value" "R2" (at 205.74 93.98 0)
+    (property "Value" "20KΩ" (at 205.74 93.98 0)
       (effects (font (size 1.27 1.27)) (justify right))
     )
@@
       (effects (font (size 1.27 1.27)) (justify right))
     )
-    (property "Value" "R2" (at 215.9 93.98 0)
+    (property "Value" "20KΩ" (at 215.9 93.98 0)
       (effects (font (size 1.27 1.27)) (justify right))
     )
@@
       (effects (font (size 1.27 1.27)))
     )
-    (property "Value" "R1" (at 218.44 100.33 90)
+    (property "Value" "10KΩ" (at 218.44 100.33 90)
       (effects (font (size 1.27 1.27)))
     )
@@
       (effects (font (size 1.27 1.27)) (justify right))
     )
-    (property "Value" "R2" (at 205.74 119.38 0)
+    (property "Value" "20KΩ" (at 205.74 119.38 0)
       (effects (font (size 1.27 1.27)) (justify right))
     )
@@
       (effects (font (size 1.27 1.27)) (justify right))
     )
-    (property "Value" "R2" (at 226.06 119.38 0)
+    (property "Value" "20KΩ" (at 226.06 119.38 0)
       (effects (font (size 1.27 1.27)) (justify right))
     )
@@
       (effects (font (size 1.27 1.27)))
     )
-    (property "Value" "R1" (at 218.44 125.73 90)
+    (property "Value" "10KΩ" (at 218.44 125.73 90)
       (effects (font (size 1.27 1.27)))
     )
@@
       (effects (font (size 1.27 1.27)) (justify right))
     )
-    (property "Value" "R2" (at 226.06 93.98 0)
+    (property "Value" "20KΩ" (at 226.06 93.98 0)
       (effects (font (size 1.27 1.27)) (justify right))
     )
@@
       (effects (font (size 1.27 1.27)) (justify right))
     )
-    (property "Value" "R2" (at 236.22 119.38 0)
+    (property "Value" "20KΩ" (at 236.22 119.38 0)
       (effects (font (size 1.27 1.27)) (justify right))
     )
@@
       (effects (font (size 1.27 1.27)))
     )
-    (property "Value" "R1" (at 208.28 100.33 90)
+    (property "Value" "10KΩ" (at 208.28 100.33 90)
       (effects (font (size 1.27 1.27)))
     )
@@
       (effects (font (size 1.27 1.27)))
     )
-    (property "Value" "R1" (at 228.6 100.33 90)
+    (property "Value" "10KΩ" (at 228.6 100.33 90)
       (effects (font (size 1.27 1.27)))
     )
@@
       (effects (font (size 1.27 1.27)))
     )
-    (property "Value" "R1" (at 228.6 125.73 90)
+    (property "Value" "10KΩ" (at 228.6 125.73 90)
       (effects (font (size 1.27 1.27)))
     )
@@
       (effects (font (size 1.27 1.27)))
     )
-    (property "Value" "R1" (at 208.28 125.73 90)
+    (property "Value" "10KΩ" (at 208.28 125.73 90)
       (effects (font (size 1.27 1.27)))
     )
@@
   )
   (symbol (lib_id "Device:R_Small") (at 233.68 92.71 180) (unit 1)
-    (in_bom yes) (on_board yes) (dnp no) (fields_autoplaced)
+    (in_bom yes) (on_board yes) (dnp no)
     (property "Reference" "R22" (at 236.22 91.44 0)
       (effects (font (size 1.27 1.27)) (justify right))
     )
-    (property "Value" "R2" (at 236.22 93.98 0)
+    (property "Value" "20KΩ" (at 236.22 93.98 0)
       (effects (font (size 1.27 1.27)) (justify right))
     )
@@
       (effects (font (size 1.27 1.27)) (justify right))
     )
-    (property "Value" "R2" (at 215.9 119.38 0)
+    (property "Value" "20KΩ" (at 215.9 119.38 0)
       (effects (font (size 1.27 1.27)) (justify right))
     )
@@
       (effects (font (size 1.27 1.27)))
     )
-    (property "Value" "R2" (at 198.12 125.73 90)
+    (property "Value" "20KΩ" (at 198.12 125.73 90)
       (effects (font (size 1.27 1.27)))
     )
