File: Kicad/mainboard/v1b/memory.kicad_sch (KiCad schematic)
At the start: 11 parts, among them U26 74HC00, U27 74HC85, U28 62256, U29 SST39SF

Commit message: v2a update
Connections:
- net A15: now also U26.13
- net at U27.5 (Oa>b): no longer U26.13
- no-connect marks 0 -> 1
Changed lines of the file:
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@@
   (junction (at 39.37 124.46) (diameter 0) (color 0 0 0 0)
   )
+  (no_connect (at 50.8 72.39))
   (wire (pts (xy 39.37 124.46) (xy 52.07 124.46))
     (stroke (width 0) (type default))
@@
     (stroke (width 0) (type default))
   )
-  (wire (pts (xy 50.8 72.39) (xy 59.69 72.39))
-    (stroke (width 0) (type default))
-  )
   (wire (pts (xy 52.07 124.46) (xy 64.77 124.46))
     (stroke (width 0) (type default))
@@
     (property "Intersheetrefs" "${INTERSHEET_REFS}" (at 137.386 57.15 0)
       (effects (font (size 1.27 1.27)) (justify left) hide)
+    )
+  )
+  (global_label "A15" (shape input) (at 59.69 72.39 180) (fields_autoplaced)
+    (effects (font (size 1.27 1.27)) (justify right))
+    (property "Intersheetrefs" "${INTERSHEET_REFS}" (at 53.1972 72.39 0)
+      (effects (font (size 1.27 1.27)) (justify right) hide)
     )
   )
@@
   )
   (symbol (lib_id "74xx:74HC00") (at 67.31 85.09 0) (unit 3)
-    (in_bom yes) (on_board yes) (dnp no) (fields_autoplaced)
+    (in_bom yes) (on_board yes) (dnp no)
     (property "Reference" "U26" (at 67.3017 76.2 0)
       (effects (font (size 1.27 1.27)))
