File: Kicad/mainboard/v1b/v1b.kicad_sch (KiCad schematic)
At the start: 12 parts, among them U1 65c02

Commit message: big v1b commit
Parts:
- removed H1, H2, H3, H4: MountingHole, MountingHole:MountingHole_3.2mm_M3_ISO14580, symbol Mechanical:MountingHole
- added H? (x4): MountingHole_Pad, MountingHole:MountingHole_3.2mm_M3_ISO14580_Pad, symbol Mechanical:MountingHole_Pad
- added TP1, TP2, TP3, TP4: TestPoint, TestPoint:TestPoint_Pad_2.0x2.0mm, symbol Connector:TestPoint
Connections:
- net +5V: now also TP1.1
- net GND: now also H?.1, H?.1, H?.1, H?.1, TP2.1
- net ~{RESET}: now also TP3.1
- net ø2: now also TP4.1
Other:
- moved on the sheet: SY1

Commit message: v2a update
Parts:
- added R44: 3.3kΩ, Resistor_THT:R_Axial_DIN0204_L3.6mm_D1.6mm_P7.62mm_Horizontal, symbol Device:R_Small
- gave numbers to parts that had none: 4
Connections:
- net +5V: now also R44.2
- net at U1.4 (ϕ1): now also R44.1
- no-connect marks 4 -> 3
Changed lines of the file:
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@@
   (junction (at 48.26 15.24) (diameter 0) (color 0 0 0 0)
   )
-  (no_connect (at 35.56 34.29))
   (no_connect (at 35.56 77.47))
   (no_connect (at 35.56 36.83))
   (no_connect (at 35.56 72.39))
+  (wire (pts (xy 29.21 34.29) (xy 30.48 34.29))
+    (stroke (width 0) (type default))
+  )
   (wire (pts (xy 25.4 64.77) (xy 35.56 64.77))
     (stroke (width 0) (type default))
   )
+  (wire (pts (xy -12.7 97.79) (xy -7.62 97.79))
+    (stroke (width 0) (type default))
+  )
   (wire (pts (xy 48.26 15.24) (xy 50.8 15.24))
     (stroke (width 0) (type default))
@@
     )
   )
+  (symbol (lib_id "power:+5V") (at 29.21 34.29 90) (unit 1)
+    (in_bom yes) (on_board yes) (dnp no) (fields_autoplaced)
+    (property "Reference" "#PWR0179" (at 33.02 34.29 0)
+      (effects (font (size 1.27 1.27)) hide)
+    )
+    (property "Value" "+5V" (at 25.4 34.29 90)
+      (effects (font (size 1.27 1.27)) (justify left))
+    )
+    (property "Footprint" "" (at 29.21 34.29 0)
+      (effects (font (size 1.27 1.27)) hide)
+    )
+    (property "Datasheet" "" (at 29.21 34.29 0)
+      (effects (font (size 1.27 1.27)) hide)
+    )
+    (pin "1")
+    (instances
+      (project "v1b"
+        (path "/82bc3382-6295-4121-a2db-2433a00f189b"
+          (reference "#PWR0179") (unit 1)
+        )
+      )
+    )
+  )
   (symbol (lib_id "power:+5V") (at 48.26 15.24 90) (unit 1)
     (in_bom yes) (on_board yes) (dnp no) (fields_autoplaced)
@@
   (symbol (lib_id "Mechanical:MountingHole_Pad") (at 45.085 116.205 0) (unit 1)
     (in_bom yes) (on_board yes) (dnp no) (fields_autoplaced)
-    (property "Reference" "H?" (at 48.26 113.665 0)
+    (property "Reference" "H2" (at 48.26 113.665 0)
       (effects (font (size 1.27 1.27)) (justify left))
     )
@@
       (project "v1b"
         (path "/82bc3382-6295-4121-a2db-2433a00f189b"
-          (reference "H?") (unit 1)
+          (reference "H2") (unit 1)
         )
       )
@@
   (symbol (lib_id "Mechanical:MountingHole_Pad") (at 21.59 126.365 0) (unit 1)
     (in_bom yes) (on_board yes) (dnp no) (fields_autoplaced)
-    (property "Reference" "H?" (at 24.765 123.825 0)
+    (property "Reference" "H3" (at 24.765 123.825 0)
       (effects (font (size 1.27 1.27)) (justify left))
     )
@@
       (project "v1b"
         (path "/82bc3382-6295-4121-a2db-2433a00f189b"
-          (reference "H?") (unit 1)
+          (reference "H3") (unit 1)
         )
       )
@@
   (symbol (lib_id "Mechanical:MountingHole_Pad") (at 45.085 126.365 0) (unit 1)
     (in_bom yes) (on_board yes) (dnp no) (fields_autoplaced)
-    (property "Reference" "H?" (at 48.26 123.825 0)
+    (property "Reference" "H4" (at 48.26 123.825 0)
       (effects (font (size 1.27 1.27)) (justify left))
     )
@@
       (project "v1b"
         (path "/82bc3382-6295-4121-a2db-2433a00f189b"
-          (reference "H?") (unit 1)
+          (reference "H4") (unit 1)
         )
       )
@@
   (symbol (lib_id "Mechanical:MountingHole_Pad") (at 21.59 116.205 0) (unit 1)
     (in_bom yes) (on_board yes) (dnp no) (fields_autoplaced)
-    (property "Reference" "H?" (at 24.765 113.665 0)
+    (property "Reference" "H1" (at 24.765 113.665 0)
       (effects (font (size 1.27 1.27)) (justify left))
     )
@@
       (project "v1b"
         (path "/82bc3382-6295-4121-a2db-2433a00f189b"
-          (reference "H?") (unit 1)
+          (reference "H1") (unit 1)
         )
       )
@@
         )
       )
+    )
+  )
+  (symbol (lib_id "Device:R_Small") (at 33.02 34.29 270) (unit 1)
+    (in_bom yes) (on_board yes) (dnp no)
+    (property "Reference" "R44" (at 33.02 31.75 90)
+      (effects (font (size 1.27 1.27)) (justify right))
+    )
+    (property "Value" "3.3kΩ" (at 35.56 36.83 90)
+      (effects (font (size 1.27 1.27)) (justify right))
+    )
+    (property "Footprint" "Resistor_THT:R_Axial_DIN0204_L3.6mm_D1.6mm_P7.62mm_Horizontal" (at 33.02 34.29 0)
+      (effects (font (size 1.27 1.27)) hide)
+    )
+    (property "Datasheet" "~" (at 33.02 34.29 0)
+      (effects (font (size 1.27 1.27)) hide)
+    )
+    (pin "1")
+    (pin "2")
+    (instances
+      (project "v1b"
+        (path "/82bc3382-6295-4121-a2db-2433a00f189b"
+          (reference "R44") (unit 1)
+        )
+      )
