File: Kicad/mainboard/v1b/video.kicad_sch (KiCad schematic)
At the start: 30 parts, among them U10 74HC590A, U11 74HC590A, U12 74HC574, U13 74HC165, U14 74HC157, U15 74HC574, U7 74HC138, U8 SST39SF, U9 74HC574

Commit message: big v1b commit
Parts:
- removed JP1: SolderJumper_3_Open, Jumper:SolderJumper-3_P1.3mm_Open_Pad1.0x1.5mm, symbol Jumper:SolderJumper_3_Open
- U10, U11: value 74HC590A -> 74HC590
Connections:
- net ~{VPixel} is gone; now on net BusDriver: U10.12 (~{CE}), U9.1 (OE)
- net ~{RegTick}: now also U10.11 (CPC), U11.11 (CPC), U7.13 (~{Y2})
- removed net ~{CharTick}: U10.11 (CPC), U11.11 (CPC), U7.15 (~{Y0})
- no-connect marks 12 -> 13
Other:
- moved on the sheet: U13
